File: pcb/pcb.kicad_pcb (KiCad board)
At the start: 2 copper layers, 0 parts

Commit message: pcb update
Routing:
- net (no net): track 558.8 -> 821.7 mm, vias 50 -> 99

Commit message: updates
Routing:
- net (no net): track 821.7 -> 315.0 mm, vias 99 -> 50
Other:
- board text removed: "10k"
- board text removed: "433"
- board text removed: "pot"
- board text removed: "sleep"
- board text removed: "tog"
